File: DMG-KGDU-MOD/DMG-KGDU-MOD.kicad_pcb (KiCad board)
At the start: 2 copper layers, 51 x 60.7 mm, 23 parts, among them U0 CartBus, U1 PRG, U2 MBC3A, U3 RAM, U4 MM1134, U5 74LVC1G32, X1 Crystal_D2mm_L6mm_Horizontal

Commit message: A02-MOD and REV2 KGDU
Other:
- board text added: "F-RAM MOD BOARD REV2"
- board text added: "RDM 202301"
- board text removed: "F-ROM MOD BOARD REV1"
- board text removed: "RDM 2023"
Changed lines of the file:
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@@
     (effects (font (size 0.8 0.8) (thickness 0.2)) (justify mirror))
   )
-  (gr_text "F-ROM\nMOD BOARD\nREV1" (at 175.26 59.944) (layer "B.Mask")
+  (gr_text "F-RAM\nMOD BOARD\nREV2" (at 175.26 59.944) (layer "B.Mask")
     (effects (font (size 0.7 0.7) (thickness 0.1)) (justify mirror))
   )
@@
     (effects (font (size 0.75 0.75) (thickness 0.15)) (justify mirror))
   )
-  (gr_text "RDM 2023" (at 146.05 59.055) (layer "B.Mask")
-    (effects (font (size 1 1) (thickness 0.25)) (justify mirror))
+  (gr_text "RDM 202301" (at 151.383127 59.072312) (layer "B.Mask")
+    (effects (font (size 1 1) (thickness 0.25)) (justify left mirror))
   )
   (gr_text "7" (at 172.466 64.897) (layer "B.Mask")
