File: DMG-KGDU-MOD2/DMG-KGDU-MOD2.kicad_pcb (KiCad board)
At the start: 2 copper layers, 51 x 60.7 mm, 23 parts, among them U0 CartBus, U1 PRG, U2 MBC3A, U3 RAM, U4 MM1134, U5 74LVC1G32, X1 Crystal_D2mm_L6mm_Horizontal

Commit message: A02-MOD and REV2 KGDU
Other:
- board text added: "F-RAM/BATT MOD BOARD REV2"
- board text removed: "F-ROM/BATT MOD BOARD REV1"
Changed lines of the file:
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@@
     (effects (font (size 0.8 0.8) (thickness 0.2)) (justify mirror))
   )
-  (gr_text "F-ROM/BATT\nMOD BOARD\nREV1" (at 175.26 60.071) (layer "B.Mask")
+  (gr_text "F-RAM/BATT\nMOD BOARD\nREV2" (at 175.26 60.071) (layer "B.Mask")
     (effects (font (size 0.7 0.7) (thickness 0.1)) (justify mirror))
   )

Commit message: Update for new stuff.
Parts:
- U5: footprint Package_SO:TSOP-6_1.65x3.05mm_P0.95mm -> Package_TO_SOT_SMD:SOT-23-5_HandSoldering
Routing:
- net VCC: track 158.8 -> 88.6 mm
- net GND: track 50.5 -> 16.4 mm
- net VBATT: track 43.1 -> 35.5 mm
- net VOUT: track 49.4 -> 44.5 mm
- net BT+: track 84.5 -> 84.0 mm
Other:
- board text added: "DMG-KGDU-M2"
- board text added: "F-RAM/BATT MOD R3"
- board text added: "RDM 2023OCT26"
- board text removed: "DMG-KGDU-MOD2"
- board text removed: "F-RAM/BATT MOD BOARD REV2"
- board text removed: "RDM 202301"
